File: pcb_design/microcontrolador.kicad_sch (KiCad schematic)
At the start: 28 parts, among them SW1 SMD_6.2x6.2mm_h7.0mm, U5 ESP32-S3-WROOM-1(N16R8), U6 TYPE-C 16PLT-H10.0

Commit message: rediseno de esquematicos, rediseno de enrutado de pcb, eleccion de componentes basics
Parts:
- removed C10: 10uF, PCM_Capacitor_SMD_AKL:C_0805_2012Metric, symbol PCM_Capacitor_AKL:C_0805
- removed C3: 1uF, Capacitor_SMD_AKL:C_0603_1608Metric, symbol PCM_Capacitor_US_AKL:C_0603
- removed D11, D12, D13: Red, SparkFun-LED:LED_0603_1608Metric_Red, symbol SparkFun-LED:LED_Red_0603
- removed D14: B0540LW, PCM_Diode_SMD_AKL:D_SOD-123, symbol PCM_Diode_Schottky_AKL:B0540LW
- removed D15, D16: ESD5B5.0S, PCM_Diode_SMD_AKL:D_SOD-523, symbol PCM_Diode_TVS_AKL:ESD5B5.0S
- removed D8: PESD3V3L1BA, Diode_SMD_AKL:D_SOD-323_TVS, symbol PCM_Diode_TVS_AKL:PESD3V3L1BA
- removed H5, H6, H7, H8: MountingHole, MountingHole:MountingHole_2.2mm_M2, symbol Mechanical:MountingHole
- removed R10: 10k, Resistor_SMD_AKL:R_0603_1608Metric, symbol PCM_Resistor_US_AKL:R_0603
- removed R11: 4.7K, Resistor_SMD_AKL:R_0603_1608Metric, symbol PCM_Resistor_US_AKL:R_0603
- removed R12, R13: 4.7k, EasyEDA:R0603, symbol EasyEDA:RC0603FR-074K7L
- removed R18: 5.1K, PCM_Resistor_SMD_AKL:R_0603_1608Metric, symbol PCM_Resistor_US_AKL:R_0603
- removed R19, R20: 33R, PCM_Resistor_SMD_AKL:R_0603_1608Metric, symbol PCM_Resistor_US_AKL:R_0603
- removed SW1: SMD_6.2x6.2mm_h7.0mm, PCM_SparkFun-Switch:Push_SMD_6.2x6.2mm, symbol PCM_SparkFun-Switch:SPST_Push_SMD_6.2x6.2mm_h7.0mm
- removed TP2: TestPoint_Hole1, 4ms_TestPoint:TestPoint_WireHole, symbol MG_ELECTROMECANICAL:TestPoint_Hole1
- removed U5: ESP32-S3-WROOM-1(N16R8), EasyEDA:WIRELM-SMD_ESP32-S3-WROOM-1, symbol EasyEDA:ESP32-S3-WROOM-1(N16R8)
- removed U6: TYPE-C 16PLT-H10.0, EasyEDA:TYPE-C-SMD_USB4120-03-C, symbol EasyEDA:TYPE-C16PLT-H10.0
- added C1: 10uF 10V, EasyEDA:C0603, symbol EasyEDA:CC0603KRX7R6BB105
- added C2: 10uF, PCM_Capacitor_SMD_AKL:C_0805_2012Metric, symbol PCM_Capacitor_AKL:C_0805
- added C22: 10uF 50v, EasyEDA:C0805, symbol EasyEDA:GRM21BR61H106KE43L
- added C23: 100nF 50V, EasyEDA:C0603, symbol EasyEDA:CC0603KRX7R9BB104
- added C24: 1uF 50V, EasyEDA:C0805, symbol EasyEDA:CL21B105KBFNNNE
- added D1: PESD3V3L1BA_C22466620, EasyEDA:SOD-323_L1.7-W1.3-LS2.6-BI, symbol EasyEDA:PESD3V3L1BA_C22466620
- added D6: B0540LW, PCM_Diode_SMD_AKL:D_SOD-123, symbol PCM_Diode_Schottky_AKL:B0540LW
- added D7, D8: ESD5B5.0S, PCM_Diode_SMD_AKL:D_SOD-523, symbol PCM_Diode_TVS_AKL:ESD5B5.0S
- added H1, H2, H3, H4: MountingHole, MountingHole:MountingHole_2.2mm_M2, symbol Mechanical:MountingHole
- added L1: 220 @100MHZ 3A, EasyEDA:L0805, symbol EasyEDA:MPZ2012S221AT000
- added R13, R19: 4.7k 100mW, EasyEDA:R0603, symbol EasyEDA:RCA034K7JLF
- added R18, R21: 10K 125mW, EasyEDA:R0805, symbol EasyEDA:0805W8F1002T5E
- added SW2: KMR221GLFS, EasyEDA:KEY-SMD_KMR2XXGXXX, symbol EasyEDA:KMR221GLFS
- added TP1: TestPoint_Hole1, 4ms_TestPoint:TestPoint_WireHole, symbol MG_ELECTROMECANICAL:TestPoint_Hole1
- added U1: ESP32-S3-WROOM-1(N16R8), EasyEDA:WIRELM-SMD_ESP32-S3-WROOM-1, symbol EasyEDA:ESP32-S3-WROOM-1(N16R8)
- added USB1: USB-TYPE-C-018, EasyEDA:USB-C_SMD-TYPE-C-31-M-12, symbol EasyEDA:USB-TYPE-C-018
- R14: value 560 -> 5.1K; footprint Resistor_SMD_AKL:R_0603_1608Metric -> PCM_Resistor_SMD_AKL:R_0603_1608Metric; LCSC Part C114629 -> C105580
- R15: value 220 -> 5.1K; footprint Resistor_SMD_AKL:R_0603_1608Metric -> PCM_Resistor_SMD_AKL:R_0603_1608Metric; LCSC Part C107696 -> C105580
- R16: value 10k -> 33R; LCSC Part C98220 -> C126353
- R17: value 5.1K -> 33R; LCSC Part C105580 -> C126353
Connections:
- net +3.3V: now also D1.2, L1.1, R18.2, R21.2; no longer R15.1, R16.1
- net BOOT: now also R18.1, SW2.1, SW2.2, U1.27 (IO0); no longer R16.2
- net EN: now also C1.2, R21.1, U1.3 (EN)
- net GND: now also R14.2, R15.2, C1.1, C2.2, C22.2, C23.2, C24.2, D1.1, D7.1 (K), D8.1 (K), R13.1, R19.1, SW2.3, SW2.4, U1.1 (GND), U1.40 (GND), U1.41 (GND), USB1.0 (SH), USB1.1 (SH), USB1.2 (SH), USB1.3 (SH), USB1.A1 (GND), USB1.A12 (GND), USB1.B1 (GND), USB1.B12 (GND); no longer R17.2
- net USB_D+: now also R17.2, D8.2 (A), U1.14 (IO20)
- net USB_D-: now also R16.2, D7.2 (A), U1.13 (IO19)
- net VBUS: now also C2.1, D6.2 (A), TP1.1, USB1.A4 (VBUS), USB1.A9 (VBUS), USB1.B4 (VBUS), USB1.B9 (VBUS)
- net VCC: now also D6.1 (K)
- net at R17.1: now also USB1.A6 (DP1), USB1.B6 (DP2)
- net +5V: no longer names the net of R14.1
- net +5V: now also USB1.A5 (CC1)
- new net: R13.2, U1.16 (IO46)
- new net: R16.1, USB1.A7 (DN1), USB1.B7 (DN2)
- new net: R15.1, USB1.B5 (CC2)
- new net: C22.1, C23.1, C24.1, L1.2, U1.2 (3V3)
- new net: R19.2, U1.26 (IO45)
- no-connect marks 13 -> 8
