File: pcb_design/pcb_design.kicad_sch (KiCad schematic)
At the start: 91 parts, among them J1 PINHD_1x9_Female, J11 DB128L-5.08-2P-BK-S, J12 PINHD_1x4_Female, J2 PINHD_1x10_Female, J3 DB128L-5.08-2P-BK-S, J4 PINHD_1x3_Female, J5 PINHD_1x4_Female, Q11 MMUN2211LT1G, Q12 AO3401A, Q5 MMUN2211LT1G, Q6 AO3401A, Q7 MMUN2211LT1G, Q8 AO3401A, Q9 MMUN2211LT1G, SW1 KMR221GLFS, U1 L78M05CDT, U2 ESP32-S3-WROOM-1(N16R8), U3 L78M05CDT, U4 L78M05CDT

Commit message: terminacion de enrutado pcb de 4 capas, cambios en la huella de usb  y mountain hole capa de potencia solo para lineas delgadas de alimentacion, posible cambio para servo de 20kg
Connections:
- net GPIO35: now also J2.5; no longer J2.4
- net GPIO36: now also J2.4; no longer J2.5
Changed lines of the file:
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@@
 	(wire
 		(pts
+			(xy 88.9 370.84) (xy 107.95 370.84)
+		)
+		(stroke
+			(width 0)
+			(type default)
+		)
+	)
+	(wire
+		(pts
 			(xy 424.18 153.67) (xy 424.18 156.21)
 		)
@@
 	(wire
 		(pts
+			(xy 88.9 368.3) (xy 107.95 368.3)
+		)
+		(stroke
+			(width 0)
+			(type default)
+		)
+	)
+	(wire
+		(pts
 			(xy 137.16 29.21) (xy 147.32 29.21)
 		)
@@
 	(wire
 		(pts
-			(xy 88.9 370.84) (xy 107.95 370.84)
-		)
-		(stroke
-			(width 0)
-			(type default)
-		)
-	)
-	(wire
-		(pts
 			(xy 335.28 292.1) (xy 335.28 289.56)
 		)
@@
 	(wire
 		(pts
-			(xy 88.9 368.3) (xy 107.95 368.3)
-		)
-		(stroke
-			(width 0)
-			(type default)
-		)
-	)
-	(wire
-		(pts
 			(xy 534.67 27.94) (xy 537.21 27.94)
 		)
@@
 	)
 	(label "GPIO36"
-		(at 88.9 370.84 0)
+		(at 88.9 368.3 0)
 		(effects
 			(font
@@
 	)
 	(label "GPIO35"
-		(at 88.9 368.3 0)
+		(at 88.9 370.84 0)
 		(effects
 			(font
